File: Electronics/controller/controller.kicad_pcb (KiCad board)
At the start: 2 copper layers, 78.3 x 90 mm, 58 parts, among them J1 Xlim, J10 GPIO_BRIDGE, J11 X Axis, J12 Y Axis, J13 Z Axis, J14 USB_A, J2 Zlim, J3 Ylim, J4 estop, J5 Vin, J6 Screw_Terminal_01x05, J8 GPIO_MCU, J9 ICSP, SW1 SW_DIP_x08, U1 ULN2003A, U2 Mini360, U3 ATmega328P-A, U4 MCP2221AxSL, U5 Bluetooth, Y1 16MHz

Commit message: added board gerbers
Other:
- board text added: "CNC Controller X.B. 08/23 rev A"
- board text added: "JLCJLCJLCJLC"
Changed lines of the file:
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@@
     )
   )
-  (gr_rect (start 66.7 78.6) (end 75.7 81.4)
+  (gr_rect (start 66.2 78.5) (end 79.2 81.7)
     (stroke (width 0.15) (type solid)) (fill solid) (layer "B.SilkS"))
   (gr_line (start 62.25 94.5) (end 71.260419 94.5)
@@
   (gr_arc (start 113.280419 106) (mid 111.815953 109.535534) (end 108.280419 111)
     (stroke (width 0.1) (type default)) (layer "Edge.Cuts"))
+  (gr_text "JLCJLCJLCJLC" (at 88.4 83.8) (layer "B.SilkS")
+    (effects (font (size 1 1) (thickness 0.15)) (justify left bottom mirror))
+  )
+  (gr_text "CNC Controller\nX.B. 08/23\nrev A" (at 88.6 81.4) (layer "B.SilkS")
+    (effects (font (size 2.2 2.2) (thickness 0.4) bold) (justify left bottom mirror))
+  )
   (gr_text "B' A' A B" (at 112 82 90) (layer "B.SilkS")
     (effects (font (size 1.3 1.3) (thickness 0.2)) (justify left bottom mirror))
